Commit message: Add files via upload

File: dualarm_config/urdf/dualarm.urdf (robot description, URDF)
Before this commit: robot dualarm, 19 links, 18 joints
Links:
- added link mani2_link1, mass 0.67076; collision mesh filename=package://dualarm_config/meshes/mani2_link1.STL; visual mesh filename=package://dualarm_config/meshes/mani2_link1.STL
- link base_link: geometry collision mesh filename=package://dualarm_config/meshes/base.STL; visual mesh filename=package://dualarm_config/meshes/base.STL
- link mani1_eff: mass 0.264591621524854 -> 0.26908; geometry collision mesh filename=package://dualarm_config/meshes/mani1_eef.STL; visual mesh filename=package://dualarm_config/meshes/mani1_eef.STL
- link mani2_base: mass 1.0280663793568 -> 0.43725
- link mani2_link2: mass 0.53869 -> 0.63538
- link mani2_link3: mass 0.5456 -> 0.55009
- link mani2_link4: mass 0.38216 -> 0.45928
- link mani2_link5: mass 0.34477 -> 0.43981
- link mani2_link6: mass 0.25794 -> 0.30699
- link mani2_link7: mass 0.085765 -> 0.10158
- link mani2_link8: mass 0.280769723735081 -> 0.26908; geometry collision mesh filename=package://dualarm_config/meshes/mani2_eef.STL; visual mesh filename=package://dualarm_config/meshes/mani2_eef.STL
Joints:
- added joint mani2_fixed: type fixed, parent mani2_base, child mani2_link1, origin xyz=0 0 0.012 rpy=0 0 1.5708, axis 0 0 0
- joint base_joint_left: origin xyz=0.23 0 0.112 rpy=0 0 0 -> xyz=0.230 0 0.376 rpy=0 0 0
- joint base_joint_right: origin xyz=-0.23 0 0.112 rpy=0 0 0 -> xyz=-0.230 0 0.364 rpy=0 0 0
- joint mani1_joint7: origin xyz=0 -0.3209 0 rpy=1.5708 0 0 -> xyz=0 -0.175 0.0 rpy=1.5708 0 0
- joint mani2_joint1: origin xyz=0 0 0.1125 rpy=6.123E-17 0 0 -> xyz=0 0 0.125 rpy=0 0 1.5708; parent mani2_base -> mani2_link1
- joint mani2_joint2: origin xyz=0 0 0.08 rpy=-1.5708 -1.2246E-16 1.4997E-32 -> xyz=0 -0.069 0.0675 rpy=-1.5708 0 0
- joint mani2_joint3: origin xyz=0 -0.211 0 rpy=1.5708 0 1.2246E-16 -> xyz=0 -0.2197 0.069 rpy=1.5708 0 0
- joint mani2_joint4: origin xyz=0 0 0.089 rpy=-1.5708 1.2246E-16 -1.4997E-32 -> xyz=0 -0.061 0.0753 rpy=-1.5708 0 0
- joint mani2_joint5: origin xyz=0 -0.192 0 rpy=1.5708 0 -1.2246E-16 -> xyz=0 -0.2 0.061 rpy=-1.5708 0 3.1416
- joint mani2_joint6: axis 0 0 1 -> 0 0 -1; origin xyz=0 0 0.258 rpy=-1.5708 1.2246E-16 1.4997E-32 -> xyz=0 0.032 0.25 rpy=-1.5708 0 0
- joint mani2_joint7: origin xyz=0 -0.1745 0 rpy=1.5708 0 -1.2246E-16 -> xyz=0 -0.0405 -0.032 rpy=1.5708 0 0
