Commit message: Add files via upload

File: dualarm_config/urdf/dualarm_before_220610.urdf (robot description, URDF)
Before this commit: robot dualarm, 23 links, 22 joints
Links:
- removed link camera
- removed link lidar1
- removed link table
- link mani1_eff: geometry collision mesh filename=package://dualarm_config/meshes/mani1_eef.STL; visual mesh filename=package://dualarm_config/meshes/mani1_eef.STL
- link mani1_link2: geometry collision mesh filename=package://dualarm_config/meshes/mani1_link2.STL; visual mesh filename=package://dualarm_config/meshes/mani1_link2.STL
- link mani1_link3: geometry collision mesh filename=package://dualarm_config/meshes/mani1_link3.STL; visual mesh filename=package://dualarm_config/meshes/mani1_link3.STL
- link mani1_link4: geometry collision mesh filename=package://dualarm_config/meshes/mani1_link4.STL; visual mesh filename=package://dualarm_config/meshes/mani1_link4.STL
- link mani1_link5: geometry collision mesh filename=package://dualarm_config/meshes/mani1_link5.STL; visual mesh filename=package://dualarm_config/meshes/mani1_link5.STL
- link mani1_link6: geometry collision mesh filename=package://dualarm_config/meshes/mani1_link6.STL; visual mesh filename=package://dualarm_config/meshes/mani1_link6.STL
- link mani1_link7: geometry collision mesh filename=package://dualarm_config/meshes/mani1_link7.STL; visual mesh filename=package://dualarm_config/meshes/mani1_link7.STL
- link mani2_link7: geometry collision mesh filename=package://dualarm_config/meshes/mani2_link7.STL; visual mesh filename=package://dualarm_config/meshes/mani2_link7.STL
Joints:
- removed joint camera_joint
- removed joint lidar1_joint
- removed joint table_joint
